Commit message: rename: prefix klaus to kls

File: urdf/workspace.urdf.xacro (robot description, xacro)
@@ -2,5 +2,5 @@
 <robot xmlns:xacro="http://www.ros.org/wiki/xacro" name="workspace">
     <!-- Insert Macros -->
-    <xacro:include filename="$(find klaus_description)/urdf/workspace_macro.xacro" />
+    <xacro:include filename="$(find kls_description)/urdf/workspace_macro.xacro" />
     <!-- Parameters -->
     <xacro:arg name="prefix" default="" />

File: urdf/workspace_macro.xacro (robot description, xacro)
@@ -8,5 +8,5 @@
                 <origin xyz="0.0 0.0 0.0" rpy="0.0 0.0 0.0" />
                 <geometry>
-                    <mesh filename="package://klaus_description/meshes/visual/klaus_table.dae"
+                    <mesh filename="package://kls_description/meshes/visual/kls_table.dae"
                         scale="1.0 1.0 1.0" />
                 </geometry>
@@ -19,5 +19,5 @@
                 <geometry>
                     <mesh
-                        filename="package://klaus_description/meshes/collision/klaus_table_collision.stl"
+                        filename="package://kls_description/meshes/collision/kls_table_collision.stl"
                         scale="1.0 1.0 1.0" />
                 </geometry>
